File: Projeto.kicad_pcb (KiCad board)
At the start: 2 copper layers, 90 x 90 mm, 50 parts, among them J1 GRAVADOR, J2 PIR, J3 Conn_01x03_Socket, J4 SERIAL, J5 LDR, J6 BOTAO, J7 JUMPER, J8 JUMPER, J9 JUMPER, K1 G5LE-1, Q1 BC547, T2 Transformer_1P_1S, U1 ATmega328-P, U2 LM7805_TO220, U3 DK1203, U4 PC817C, Y1 Crystal

Commit message: zonas novas
Routing:
- net Earth: track 0.00 -> 38.6 mm
- added copper zone on B.Cu, net (none)
- removed copper zone on B.Cu, net Earth
